Commit message: add launch async

File: urdf/nubot.gazebo.xacro (robot description, xacro)
@@ -39,4 +39,62 @@
         </sensor>
     </gazebo>
+    <!-- <link name="lidar_link">
+      <inertial>
+        <origin xyz="0 0 0" rpy="0 0 0"/>
+        <mass value="0.125"/>
+        <inertia ixx="0.001" ixy="0" ixz="0" iyy="0.001" iyz="0" izz="0.001"/>
+      </inertial>
+      <collision>
+        <origin xyz="0 0 0" rpy="0 0 0"/>
+        <geometry>
+          <cylinder radius="0.0508" length="0.055"/>
+        </geometry>
+      </collision>
+      <visual>
+        <origin xyz="0 0 0" rpy="0 0 0"/>
+        <geometry>
+          <cylinder radius="0.0508" length="0.055"/>
+        </geometry>
+      </visual>
+    </link>
+    <joint name="lidar_joint" type="fixed">
+      <parent link="base_link"/>
+      <child link="lidar_link"/>
+      <origin xyz="0 0 0.12" rpy="0 0 0"/>
+    </joint>
+    <gazebo reference="lidar_link">
+      <sensor name="lidar_360" type="ray">
+        <always_on>true</always_on>
+        <visualize>true</visualize>
+        <update_rate>5</update_rate>
+        <ray>
+          <scan>
+            <horizontal>
+              <samples>360</samples>
+              <resolution>1.0</resolution>
+              <min_angle>0.0</min_angle>
+              <max_angle>6.283185</max_angle>
+            </horizontal>
+          </scan>
+          <range>
+            <min>0.12</min>
+            <max>3.5</max>
+            <resolution>0.015</resolution>
+          </range>
+          <noise>
+            <type>gaussian</type>
+            <mean>0.0</mean>
+            <stddev>0.01</stddev>
+          </noise>
+        </ray>
+        <plugin name="scan" filename="libgazebo_ros_ray_sensor.so">
+          <ros>
+            <remapping>~/out:=scan_360</remapping>
+          </ros>
+          <output_type>sensor_msgs/LaserScan</output_type>
+          <frame_name>lidar_link</frame_name>
+        </plugin>
+      </sensor>
+    </gazebo> -->
     <gazebo>
       <plugin

Commit message: pass all colcon test

File: urdf/nubot.gazebo.xacro (robot description, xacro)
@@ -39,62 +39,4 @@
         </sensor>
     </gazebo>
-    <!-- <link name="lidar_link">
-      <inertial>
-        <origin xyz="0 0 0" rpy="0 0 0"/>
-        <mass value="0.125"/>
-        <inertia ixx="0.001" ixy="0" ixz="0" iyy="0.001" iyz="0" izz="0.001"/>
-      </inertial>
-      <collision>
-        <origin xyz="0 0 0" rpy="0 0 0"/>
-        <geometry>
-          <cylinder radius="0.0508" length="0.055"/>
-        </geometry>
-      </collision>
-      <visual>
-        <origin xyz="0 0 0" rpy="0 0 0"/>
-        <geometry>
-          <cylinder radius="0.0508" length="0.055"/>
-        </geometry>
-      </visual>
-    </link>
-    <joint name="lidar_joint" type="fixed">
-      <parent link="base_link"/>
-      <child link="lidar_link"/>
-      <origin xyz="0 0 0.12" rpy="0 0 0"/>
-    </joint>
-    <gazebo reference="lidar_link">
-      <sensor name="lidar_360" type="ray">
-        <always_on>true</always_on>
-        <visualize>true</visualize>
-        <update_rate>5</update_rate>
-        <ray>
-          <scan>
-            <horizontal>
-              <samples>360</samples>
-              <resolution>1.0</resolution>
-              <min_angle>0.0</min_angle>
-              <max_angle>6.283185</max_angle>
-            </horizontal>
-          </scan>
-          <range>
-            <min>0.12</min>
-            <max>3.5</max>
-            <resolution>0.015</resolution>
-          </range>
-          <noise>
-            <type>gaussian</type>
-            <mean>0.0</mean>
-            <stddev>0.01</stddev>
-          </noise>
-        </ray>
-        <plugin name="scan" filename="libgazebo_ros_ray_sensor.so">
-          <ros>
-            <remapping>~/out:=scan_360</remapping>
-          </ros>
-          <output_type>sensor_msgs/LaserScan</output_type>
-          <frame_name>lidar_link</frame_name>
-        </plugin>
-      </sensor>
-    </gazebo> -->
     <gazebo>
       <plugin
